File: Week1/Starbie/main.kicad_pcb (KiCad board)
At the start: 2 copper layers, 100 x 88.4 mm, 7 parts, among them J1 Conn_01x04_Pin, J2 Conn_01x08_Pin, SW1 SW_Push, SW2 SW_Push, U1 DHT11, U2 XIAO-ESP32-C3-SMD

Commit message: Day 2 Complete
Parts:
- added G***: LOGO, LOGO, F.Cu at (167.0, 109.0)
- added G***: LOGO, LOGO, F.Cu at (169.5, 124.0)
- added G***: LOGO, LOGO, F.Cu at (107.0, 132.0)
Routing:
- net +3.3V: track 191.0 -> 95.4 mm
- net /SDA: track 47.1 -> 48.8 mm
- net /GPIO3: track 47.8 -> 48.9 mm
- added copper zone on F.Cu, net GND
